Commit message: first working robot

File: ros2humb_ws/src/antoniobot_description/urdf/antoniobot.urdf.xacro (robot description, xacro)
@@ -1,4 +1,5 @@
 <?xml version="1.0"?>
 <robot xmlns:xacro="http://www.ros.org/wiki/xacro" name="antoniobot">
+    <xacro:arg name="is_sim" default="true"/>
     <xacro:include filename="$(find antoniobot_description)/urdf/antoniobot_gazebo.xacro"/>
     <xacro:include filename="$(find antoniobot_description)/urdf/antoniobot_ros2_control.xacro"/>
@@ -161,4 +162,29 @@
         <origin xyz="-0.8 0.1 0" rpy="${PI/2} 0 ${PI}"/>
     </joint>
+    <!-- Virtual yaw link -->
+    <link name="virtual_yaw_link">
+        <visual>
+        <origin xyz="0 0 0" rpy="0 0 0"/>
+        <geometry>
+            <box size="0.01 0.01 0.01" />
+        </geometry>
+        </visual>
+        <inertial>
+        <origin xyz="0 0 0" />
+        <mass value="1.0e-03" />
+        <inertia ixx="1.0e-03" ixy="0.0" ixz="0.0"
+                iyy="1.0e-03" iyz="0.0"
+                izz="1.0e-03" />
+        </inertial>
+    </link>
+        <!-- Virtual yaw joint -->
+    <joint name="virtual_yaw_joint" type="revolute">
+        <limit lower="-3.1415" upper="3.1415" effort="54.0" velocity="3.14"/>
+        <parent link="gripper"/>
+        <child link="virtual_yaw_link"/>
+        <axis xyz="0 0 1"/>
+        <origin xyz="0.0 0.0 0.0" rpy="0 0 0"/>
+        <dynamics damping="0.0" friction="0.0"/>
+    </joint>
     <xacro:default_transmission number="1" />
     <xacro:default_transmission number="2" />
@@ -167,3 +193,10 @@
     <xacro:default_transmission number="5" />
     <!-- <xacro:default_transmission number="6" /> -->
+    <transmission name="transmission_6">
+        <plugin>transmission_interface/SimpleTransmission</plugin>
+        <actuator name="motor_6" role="actuator1"/>
+        <joint name="virtual_yaw_joint" role="joint1">
+            <mechanical_reduction>1.0</mechanical_reduction>
+        </joint>
+    </transmission>
 </robot>

File: ros2humb_ws/src/antoniobot_description/urdf/antoniobot_ros2_control.xacro (robot description, xacro)
@@ -12,7 +12,16 @@
             </joint>
         </xacro:macro>
-        <hardware>
-            <plugin>gazebo_ros2_control/GazeboSystem</plugin>
-        </hardware>
+        <xacro:if value="$(arg is_sim)">
+            <hardware>
+                <!-- simulated gazebo -->
+                <plugin>gazebo_ros2_control/GazeboSystem</plugin>
+            </hardware>
+        </xacro:if>
+        <xacro:unless value="$(arg is_sim)">
+            <hardware>
+                <plugin>antoniobot_controller/AntoniobotInterface</plugin>
+                <param name="port">/dev/ttyACM0</param>
+            </hardware>
+        </xacro:unless>
         <xacro:default_joint number="1" minvalue="-${PI/2}" maxvalue="${PI/2}"/>
         <xacro:default_joint number="2" minvalue="-${PI/2}" maxvalue="${PI/2}"/>
@@ -21,4 +30,11 @@
         <xacro:default_joint number="5" minvalue="-${PI/2}" maxvalue="${PI/2}"/>
         <!-- <xacro:default_joint number="6" minvalue="0" maxvalue="0.1"/> -->
+        <joint name="virtual_yaw_joint">
+            <command_interface name="position">
+                <param name="min">-3.1415</param>
+                <param name="max">3.1415</param>
+            </command_interface>
+            <state_interface name="position"/>
+        </joint>
     </ros2_control>
 </robot>

Commit message: first working branch - next integration of UI

File: ros2humb_ws/src/antoniobot_description/urdf/antoniobot.urdf.xacro (robot description, xacro)
@@ -130,5 +130,5 @@
         <origin xyz="-0.135 0.916 -0.053" rpy="0 -${PI/2} 0"/>
         <limit lower="-${PI/2}" upper="${PI/2}" velocity="${velocity}" effort="${effort}"/>
-        <axis xyz="0 1 0"/>
+        <axis xyz="0 -1 0"/>
     </joint>
     <link name="gripper_base">
@@ -152,5 +152,5 @@
         <origin xyz="0.05 0.28 -0.135" rpy="0 0 -${PI/2}"/>
         <limit lower="-${PI/2}" upper="${PI/2}" velocity="${velocity}" effort="${effort}"/>
-        <axis xyz="0 0 1"/>
+        <axis xyz="0 0 -1"/>
     </joint>
     <link name="gripper">
@@ -183,5 +183,5 @@
         <parent link="gripper"/>
         <child link="virtual_yaw_link"/>
-        <axis xyz="0 0 1"/>
+        <axis xyz="1 0 0"/>
         <origin xyz="0.0 0.0 0.0" rpy="0 0 0"/>
         <dynamics damping="0.0" friction="0.0"/>
